File: hardware/plane.kicad_pcb (KiCad board)
At the start: 2 copper layers, 32 x 100 mm, 51 parts, among them J1 USB_B_Micro, J10 Conn_01x05_Pin, J11 Conn_01x04_Pin, J2 Conn_Coaxial, J3 Conn_01x03, J4 Conn_01x03, J5 Conn_01x03, J6 Conn_01x03, J7 Conn_01x02, J8 Conn_01x03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

Commit message: add nrf24l01 connector
Parts:
- removed C19: C, Capacitor_SMD:C_0603_1608Metric
- removed J9: Conn_01x03, Connector_PinHeader_2.54mm:PinHeader_1x03_P2.54mm_Vertical
- added J12: Conn_02x04_Odd_Even, Connector_PinHeader_2.54mm:PinHeader_2x04_P2.54mm_Vertical, F.Cu at (126.3, 64.9)
- moved R5 22.5 mm to (127.2, 43.2), turned to -90 degrees
- moved D2 20.5 mm to (129.8, 45.2), turned to 180 degrees
Connections:
- U1 pad 24: SR5 -> NRF_CC
- U1 pad 31: DIO2 -> NRF_CE
- U1 pad 6: unconnected-(U1-IO34-Pad6) -> NRF_IRQ
Routing:
- net DIO2: track 87.1 -> 0.00 mm, vias 2 -> 0
- net NRF_IRQ: track 0.00 -> 41.4 mm, vias 0 -> 1
- net SR5: track 39.7 -> 0.00 mm, vias 2 -> 0
- net Net-(U1-IO23): track 26.6 -> 2.15 mm
- net NRF_CE: track 0.00 -> 23.1 mm, vias 0 -> 2
- net SCLK: track 84.6 -> 105.4 mm, vias 2 -> 4
- net NRF_CC: track 0.00 -> 16.7 mm, vias 0 -> 2
- net +5V: track 206.7 -> 194.5 mm
- net +3V3: track 162.1 -> 173.5 mm, vias 3 -> 4
- net MOSI: track 73.0 -> 79.2 mm, vias 2 -> 3
- net MISO: track 84.1 -> 86.4 mm, vias 2 -> 3
- net TX-PROG: track 103.0 -> 100.8 mm
- net LORA_RST: track 68.0 -> 70.0 mm
- net ESP32_EN: track 88.3 -> 89.1 mm
- net SR1: track 43.4 -> 44.2 mm
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Other:
- outline, holes or cut-outs redrawn
